Commit message: added effort controllers

File: franka_ros/franka_description/robots/hand backup.xacro (robot description, xacro)
@@ -35,9 +35,4 @@
         </geometry>
       </visual>
-      <collision>
-        <geometry>
-          <mesh filename="package://franka_description/meshes/collision/finger.stl"/>
-        </geometry>
-      </collision>
       <!-- for simulation -->
       <inertial>
@@ -55,10 +50,4 @@
         </geometry>
       </visual>
-      <collision>
-        <origin xyz="0 0 0" rpy="0 0 ${pi}"/>
-        <geometry>
-          <mesh filename="package://franka_description/meshes/collision/finger.stl"/>
-        </geometry>
-      </collision>
       <!-- for simulation -->
       <inertial>
@@ -84,18 +73,4 @@
       <mimic joint="${ns}_finger_joint1" />
     </joint>
-    <!-- <gazebo reference="${ns}_leftfinger">
-      <kp>10000000.0</kp>
-      <kd>1.0</kd>
-      <mu1>100000.0</mu1>
-      <mu2>100000.0</mu2>
-      <minDepth>0.001</minDepth>
-    </gazebo>
-    <gazebo reference="${ns}_rightfinger">
-      <kp>10000000.0</kp>
-      <kd>1.0</kd>
-      <mu1>100000.0</mu1>
-      <mu2>100000.0</mu2>
-      <minDepth>0.001</minDepth>
-    </gazebo> -->
   </xacro:macro>
 </robot>

File: franka_ros/franka_description/robots/panda.control.xacro (robot description, xacro)
@@ -14,4 +14,16 @@
             </transmission>
         </xacro:macro>
+        <xacro:macro name="hand_control" params="transmission joint motor">
+            <transmission name="${transmission}">
+                <type>transmission_interface/SimpleTransmission</type>
+                <joint name="${joint}">
+                    <hardwareInterface>hardware_interface/PositionJointInterface</hardwareInterface>
+                </joint>
+                <actuator name="${motor}">
+                    <hardwareInterface>hardware_interface/PosiitonJointInterface</hardwareInterface>
+                    <mechanicalReduction>1</mechanicalReduction>
+                </actuator>
+            </transmission>
+        </xacro:macro>
         <xacro:arm_control transmission="${arm_id}_tran_1" joint="${arm_id}_joint1" motor="${arm_id}_motor_1"/>
         <xacro:arm_control transmission="${arm_id}_tran_2" joint="${arm_id}_joint2" motor="${arm_id}_motor_2"/>
@@ -22,6 +34,6 @@
         <xacro:arm_control transmission="${arm_id}_tran_7" joint="${arm_id}_joint7" motor="${arm_id}_motor_7"/>
         <xacro:if value="${load_hand}">
-            <xacro:arm_control transmission="${arm_id}_leftfinger" joint="${arm_id}_finger_joint1" motor="${arm_id}_finger_joint1"/>
-            <xacro:arm_control transmission="${arm_id}_rightfinger" joint="${arm_id}_finger_joint2" motor="${arm_id}_finger_joint2"/>
+            <xacro:hand_control transmission="${arm_id}_leftfinger" joint="${arm_id}_finger_joint1" motor="${arm_id}_finger_joint1"/>
+            <xacro:hand_control transmission="${arm_id}_rightfinger" joint="${arm_id}_finger_joint2" motor="${arm_id}_finger_joint2"/>
         </xacro:if>
         <gazebo>

File: franka_ros/franka_description/robots/panda.gazebo_backup.xacro (robot description, xacro)
@@ -5,5 +5,4 @@
             <gazebo reference="${link}">
                 <material>Gazebo/White</material>
-                <implicitSpringDamper>1</implicitSpringDamper>
                 <mu1>0.2</mu1>
                 <mu2>0.2</mu2>
@@ -13,10 +12,6 @@
             <gazebo reference="${link}">
                 <material>Gazebo/Grey</material>
-                <implicitSpringDamper>1</implicitSpringDamper>
-                <kp>1000000.0</kp>
-                <kd>1.0</kd>
-                <mu1>1.0</mu1>
-                <mu2>1.0</mu2>
-                <minDepth>0.001</minDepth>
+                <mu1>0.2</mu1>
+                <mu2>0.2</mu2>
             </gazebo>
         </xacro:macro>

File: pick_and_place/urdf/objects/box.urdf (robot description, URDF)
Before this commit: robot box, 1 links, 0 joints
Links:
- link box_link: geometry collision box size=0.08 0.04 0.08; visual box size=0.08 0.04 0.08
