Commit message: added grasp plugin

File: franka_ros/franka_description/robots/panda.gazebo.xacro (robot description, xacro)
@@ -6,9 +6,20 @@
                 <material>Gazebo/White</material>
                 <implicitSpringDamper>1</implicitSpringDamper>
-                <mu1>0.2</mu1>
-                <mu2>0.2</mu2>
+                <mu1>10000.0</mu1>
+                <mu2>10000.0</mu2>
             </gazebo>
         </xacro:macro>
         <xacro:macro name="hand_gazebo" params="link">
+            <gazebo reference="${link}">
+                <material>Gazebo/Grey</material>
+                <implicitSpringDamper>1</implicitSpringDamper>
+                <kp>100000.0</kp>
+                <kd>1.0</kd>
+                <mu1>10000.0</mu1>
+                <mu2>10000.0</mu2>
+                <minDepth>0.001</minDepth>
+            </gazebo>
+        </xacro:macro>
+        <xacro:macro name="finger_gazebo" params="link">
             <gazebo reference="${link}">
                 <material>Gazebo/Grey</material>
@@ -28,9 +39,9 @@
         <xacro:arm_gazebo link="${arm_id}_link5"/>
         <xacro:arm_gazebo link="${arm_id}_link6"/>
-        <xacro:hand_gazebo link="${arm_id}_link7"/>
-        <xacro:hand_gazebo link="${arm_id}_link8"/>
+        <xacro:arm_gazebo link="${arm_id}_link7"/>
+        <xacro:arm_gazebo link="${arm_id}_link8"/>
         <xacro:hand_gazebo link="${arm_id}_hand"/>
-        <xacro:hand_gazebo link="${arm_id}_rightfinger"/>
-        <xacro:hand_gazebo link="${arm_id}_leftfinger"/>
+        <xacro:finger_gazebo link="${arm_id}_rightfinger"/>
+        <xacro:finger_gazebo link="${arm_id}_leftfinger"/>
     </xacro:macro>
 </robot>

File: franka_ros/franka_description/robots/panda_arm.xacro (robot description, xacro)
@@ -333,4 +333,21 @@
       <child link="${arm_id}_link8"/>
     </joint>
+    <gazebo>
+      <plugin name="gazebo_grasp_fix" filename="libgazebo_grasp_fix.so">
+        <arm>
+           <arm_name>panda</arm_name>
+           <palm_link> panda_link7  </palm_link>
+           <gripper_link> panda_leftfinger </gripper_link>
+           <gripper_link> panda_rightfinger </gripper_link>
+        </arm>
+       <forces_angle_tolerance>100</forces_angle_tolerance>
+       <update_rate>4</update_rate>
+       <grip_count_threshold>4</grip_count_threshold>
+       <max_grip_count>8</max_grip_count>
+       <release_tolerance>0.005</release_tolerance>
+       <disable_collisions_on_attach>false</disable_collisions_on_attach>
+       <contact_topic>__default_topic__</contact_topic>
+      </plugin>
+    </gazebo>
   </xacro:macro>
 </robot>

File: pick_and_place/urdf/objects/red_box.urdf (robot description, URDF)
Before this commit: robot red_box, 1 links, 0 joints
Links:
- link base_link: mass 0.200 -> 0.010
