Commit message: removed useless urdf and modified inertia

File: pick_and_place/urdf/objects/red_cylinder.urdf (robot description, URDF)
Before this commit: robot red_cylinder, 1 links, 0 joints
Links:
- link base_link: geometry collision cylinder length=0.08 radius=0.02; visual cylinder length=0.08 radius=0.02
