Commit message: commiting eye on hand files

File: pick_and_place/urdf/kinect.urdf (robot description, URDF)
Before this commit: robot kinect, 2 links, 1 joints
Joints:
- joint world_to_camera_joint: origin xyz=0.75 0 1.5 rpy=0 1.57 0 -> xyz=0.75 0 1.5 rpy=0 0 0

Commit message: added pose information methods

File: pick_and_place/urdf/kinect.urdf (robot description, URDF)
Before this commit: robot kinect, 2 links, 1 joints
Joints:
- joint world_to_camera_joint: origin xyz=0.75 0 1.5 rpy=0 0 0 -> xyz=0.75 0 1.5 rpy=0 1.57 0

Commit message: Changes for testing ggcnn

File: pick_and_place/urdf/kinect.urdf (robot description, URDF)
Before this commit: robot kinect, 2 links, 1 joints
Joints:
- joint world_to_camera_joint: origin xyz=0.75 0 1.5 rpy=0 1.57 0 -> xyz=0.5 0 1.0 rpy=0 1.57 0

Commit message: change fov, pipeling changes

File: pick_and_place/urdf/kinect.urdf (robot description, URDF)
Before this commit: robot kinect, 2 links, 1 joints
Joints:
- joint world_to_camera_joint: origin xyz=0.5 0 1.0 rpy=0 1.57 0 -> xyz=0.5 0 0.99 rpy=0 1.57 0
